File: SolarCarECU/SolarCarECU.sch (KiCad schematic (older format))
At the start: 112 parts, among them J1 Screw_Terminal_01x02, J2 USB_B_Micro, J3 Screw_Terminal_01x05, J4 Screw_Terminal_01x08, J5 Screw_Terminal_01x08, J6 Screw_Terminal_01x14, J7 Screw_Terminal_01x14, Q1 QM6015D, Q2 PZT2222A, Q3 QM6015D, Q4 QM6015D, Q5 QM6015D, Q6 QM6015D, U1 Teensy3.6, U10 LM324A, U2 EL7202CN, U3 EL7202CN, U4 L7805, U5 MCP2562-E-P, U6 MCP2562-E-P, U7 4504, U8 4504, U9 4504

Commit message: lots of things
Parts:
- added R48, R49, R50, R51: 4.7, Resistor_SMD:R_0603_1608Metric, symbol Device:R
- R32, R33, R34, R35, R36, R37, R38, R39, R6: value R -> 1k
- R42, R43: value R -> 0
- R8, R9: value R -> 100k
Connections:
- net +12V: now also C2.2, C3.2, C5.2, C6.2, C7.2, C8.2, Q3.3 (S), Q4.3 (S), Q5.3 (S), Q6.3 (S), U2.6 (V+), U3.6 (V+)
- net CAN0_H: now also J7.3 (Pin_3); no longer J7.2 (Pin_2)
- net CAN0_L: now also J7.2 (Pin_2); no longer J7.3 (Pin_3)
- net CAN1_H: now also J7.5 (Pin_5); no longer J7.4 (Pin_4)
- net CAN1_L: now also J7.4 (Pin_4); no longer J7.5 (Pin_5)
- net DOWN_CTRL: now also J6.10 (Pin_10); no longer J6.11 (Pin_11)
- net HAZARD_LED: now also J6.14 (Pin_14); no longer J6.10 (Pin_10)
- net KILL_SENSE: now also J6.13 (Pin_13); no longer J6.14 (Pin_14)
- net SEL_CTRL: now also J6.12 (Pin_12); no longer J6.13 (Pin_13)
- net UP_CTRL: now also J6.11 (Pin_11); no longer J6.12 (Pin_12)
- net at U3.5 (OUT_B): now also R51.2; no longer Q6.1 (G)
- net at U3.7 (OUT_A): now also R50.2; no longer Q4.1 (G)
- net at Q5.1 (G): now also R49.1; no longer U2.5 (OUT_B)
- net at Q3.1 (G): now also R48.1; no longer U2.7 (OUT_A)
- new net: Q4.1 (G), R50.1
- new net: Q6.1 (G), R51.1
- new net: R48.2, U2.7 (OUT_A)
- new net: R49.2, U2.5 (OUT_B)
Changed lines of the file:
@@
 	1    0    0    -1
 $EndComp
-Text GLabel 11550 11500 2    50   Input ~ 0
-CAN0_H
-Text GLabel 11550 11800 2    50   Input ~ 0
-CAN0_L
 $Comp
 L SolarCarECU-rescue:+3V3-power #PWR0107
@@
 P 9450 12050
 F 0 "R8" H 9520 12096 50  0000 L CNN
-F 1 "R" H 9520 12005 50  0000 L CNN
+F 1 "100k" H 9520 12005 50  0000 L CNN
 F 2 "Resistor_SMD:R_0603_1608Metric" V 9380 12050 50  0001 C CNN
 F 3 "~" H 9450 12050 50  0001 C CNN
@@
 	1    0    0    -1
 $EndComp
-Text GLabel 11500 13150 2    50   Input ~ 0
-CAN1_H
-Text GLabel 11500 13450 2    50   Input ~ 0
-CAN1_L
 $Comp
 L SolarCarECU-rescue:+3V3-power #PWR0123
@@
 P 9450 13700
 F 0 "R9" H 9520 13746 50  0000 L CNN
-F 1 "R" H 9520 13655 50  0000 L CNN
+F 1 "100k" H 9520 13655 50  0000 L CNN
 F 2 "Resistor_SMD:R_0603_1608Metric" V 9380 13700 50  0001 C CNN
 F 3 "~" H 9450 13700 50  0001 C CNN
@@
 P 3650 3150
 F 0 "R6" H 3720 3196 50  0000 L CNN
-F 1 "R" H 3720 3105 50  0000 L CNN
+F 1 "1k" H 3720 3105 50  0000 L CNN
 F 2 "Resistor_SMD:R_0603_1608Metric" V 3580 3150 50  0001 C CNN
 F 3 "~" H 3650 3150 50  0001 C CNN
@@
 Text Label 20400 7150 0    50   ~ 0
 HAZARD_CTRL
-Text Label 20400 7350 0    50   ~ 0
+Text Label 20400 7250 0    50   ~ 0
 DOWN_CTRL
-Text Label 20400 7450 0    50   ~ 0
+Text Label 20400 7350 0    50   ~ 0
 UP_CTRL
-Text Label 20400 7550 0    50   ~ 0
+Text Label 20400 7450 0    50   ~ 0
 SEL_CTRL
-Text Label 20400 7650 0    50   ~ 0
+Text Label 20400 7550 0    50   ~ 0
 KILL_SENSE
-Text Label 20400 7250 0    50   ~ 0
+Text Label 20400 7650 0    50   ~ 0
 HAZARD_LED
 Text Label 20450 3250 0    50   ~ 0
@@
 P 16950 3850
 F 0 "R32" H 17020 3896 50  0000 L CNN
-F 1 "R" H 17020 3805 50  0000 L CNN
+F 1 "1k" H 17020 3805 50  0000 L CNN
 F 2 "Resistor_SMD:R_0603_1608Metric" V 16880 3850 50  0001 C CNN
 F 3 "~" H 16950 3850 50  0001 C CNN
@@
 P 16950 4350
 F 0 "R33" H 17020 4396 50  0000 L CNN
-F 1 "R" H 17020 4305 50  0000 L CNN
+F 1 "1k" H 17020 4305 50  0000 L CNN
 F 2 "Resistor_SMD:R_0603_1608Metric" V 16880 4350 50  0001 C CNN
 F 3 "~" H 16950 4350 50  0001 C CNN
@@
 P 16950 5750
 F 0 "R34" H 17020 5796 50  0000 L CNN
-F 1 "R" H 17020 5705 50  0000 L CNN
+F 1 "1k" H 17020 5705 50  0000 L CNN
 F 2 "Resistor_SMD:R_0603_1608Metric" V 16880 5750 50  0001 C CNN
 F 3 "~" H 16950 5750 50  0001 C CNN
@@
 P 16950 6250
 F 0 "R35" H 17020 6296 50  0000 L CNN
-F 1 "R" H 17020 6205 50  0000 L CNN
+F 1 "1k" H 17020 6205 50  0000 L CNN
 F 2 "Resistor_SMD:R_0603_1608Metric" V 16880 6250 50  0001 C CNN
 F 3 "~" H 16950 6250 50  0001 C CNN
@@
 P 16950 7650
 F 0 "R36" H 17020 7696 50  0000 L CNN
-F 1 "R" H 17020 7605 50  0000 L CNN
+F 1 "1k" H 17020 7605 50  0000 L CNN
 F 2 "Resistor_SMD:R_0603_1608Metric" V 16880 7650 50  0001 C CNN
 F 3 "~" H 16950 7650 50  0001 C CNN
@@
 P 16950 8150
 F 0 "R37" H 17020 8196 50  0000 L CNN
-F 1 "R" H 17020 8105 50  0000 L CNN
+F 1 "1k" H 17020 8105 50  0000 L CNN
 F 2 "Resistor_SMD:R_0603_1608Metric" V 16880 8150 50  0001 C CNN
 F 3 "~" H 16950 8150 50  0001 C CNN
@@
 P 16950 9550
 F 0 "R38" H 17020 9596 50  0000 L CNN
-F 1 "R" H 17020 9505 50  0000 L CNN
+F 1 "1k" H 17020 9505 50  0000 L CNN
 F 2 "Resistor_SMD:R_0603_1608Metric" V 16880 9550 50  0001 C CNN
 F 3 "~" H 16950 9550 50  0001 C CNN
@@
 P 16950 10050
 F 0 "R39" H 17020 10096 50  0000 L CNN
-F 1 "R" H 17020 10005 50  0000 L CNN
+F 1 "1k" H 17020 10005 50  0000 L CNN
 F 2 "Resistor_SMD:R_0603_1608Metric" V 16880 10050 50  0001 C CNN
 F 3 "~" H 16950 10050 50  0001 C CNN
@@
 Wire Wire Line
 	10400 2500 10400 2600
-Text GLabel 21050 9000 0    50   Input ~ 0
-CAN1_H
-Text GLabel 21050 9100 0    50   Input ~ 0
-CAN1_L
-Text GLabel 21050 8800 0    50   Input ~ 0
-CAN0_H
-Text GLabel 21050 8900 0    50   Input ~ 0
-CAN0_L
 Wire Wire Line
 	21050 9100 21200 9100
@@
 $EndComp
 Wire Wire Line
-	11500 13150 11200 13150
-Wire Wire Line
 	10900 13150 10900 13200
 Wire Wire Line
@@
 	10750 13400 10900 13400
 Connection ~ 11200 13450
-Wire Wire Line
-	11200 13450 11500 13450
 $Comp
 L SolarCarECU-rescue:R-Device R11
@@
 $EndComp
 Wire Wire Line
-	11550 11500 11250 11500
-Wire Wire Line
 	10950 11500 10950 11550
 Connection ~ 11250 11500
@@
 Connection ~ 11250 11800
 Wire Wire Line
-	11250 11800 11550 11800
-Wire Wire Line
 	10750 11750 10950 11750
 Wire Wire Line
@@
 	6250 8250 6250 8500
 Wire Wire Line
-	5750 8700 6700 8700
-Wire Wire Line
 	6500 8400 5800 8400
 Wire Wire Line
@@
 	5350 7950 5800 7950
 Wire Wire Line
-	5750 8500 6250 8500
-Wire Wire Line
 	5800 7950 6050 7950
 Wire Wire Line
@@
 	6250 5950 6250 6200
 Wire Wire Line
-	5750 6400 6700 6400
-Wire Wire Line
 	6500 6100 5800 6100
 Wire Wire Line
@@
 	5350 5650 5800 5650
 Wire Wire Line
-	5750 6200 6250 6200
-Wire Wire Line
 	5800 5650 6050 5650
 Wire Wire Line
@@
 P 4700 2250
 F 0 "R43" H 4770 2296 50  0000 L CNN
-F 1 "R" H 4770 2205 50  0000 L CNN
+F 1 "0" H 4770 2205 50  0000 L CNN
 F 2 "Resistor_SMD:R_0603_1608Metric" V 4630 2250 50  0001 C CNN
 F 3 "~" H 4700 2250 50  0001 C CNN
@@
 P 4200 2250
 F 0 "R42" H 4270 2296 50  0000 L CNN
-F 1 "R" H 4270 2205 50  0000 L CNN
+F 1 "0" H 4270 2205 50  0000 L CNN
 F 2 "Resistor_SMD:R_0603_1608Metric" V 4130 2250 50  0001 C CNN
 F 3 "~" H 4200 2250 50  0001 C CNN
@@
 Text Label 5250 10700 0    50   ~ 0
 LV_MOTOR_L_REV_EN
+$Comp
+L power:+12V #PWR0169
+U 1 1 5CA2EE3B
+P 4550 5650
+F 0 "#PWR0169" H 4550 5500 50  0001 C CNN
+F 1 "+12V" H 4565 5823 50  0000 C CNN
+F 2 "" H 4550 5650 50  0001 C CNN
+F 3 "" H 4550 5650 50  0001 C CNN
+	1    4550 5650
+	1    0    0    -1
+$EndComp
+Wire Wire Line
+	4550 5650 4900 5650
+Connection ~ 4900 5650
+$Comp
+L power:+12V #PWR0170
+U 1 1 5CA822B5
+P 4550 7950
+F 0 "#PWR0170" H 4550 7800 50  0001 C CNN
+F 1 "+12V" H 4565 8123 50  0000 C CNN
+F 2 "" H 4550 7950 50  0001 C CNN
+F 3 "" H 4550 7950 50  0001 C CNN
+	1    4550 7950
+	1    0    0    -1
+$EndComp
+Wire Wire Line
+	4550 7950 4900 7950
+Connection ~ 4900 7950
+$Comp
+L Device:R R48
+U 1 1 5CAD66BD
+P 6000 6200
+F 0 "R48" V 6100 6100 50  0000 C CNN
+F 1 "4.7" V 6100 6300 50  0000 C CNN
+F 2 "Resistor_SMD:R_0603_1608Metric" V 5930 6200 50  0001 C CNN
+F 3 "~" H 6000 6200 50  0001 C CNN
+	1    6000 6200
+	0    1    1    0
+$EndComp
+$Comp
+L Device:R R49
+U 1 1 5CAD6840
+P 6000 6400
+F 0 "R49" V 6100 6300 50  0000 C CNN
+F 1 "4.7" V 6100 6500 50  0000 C CNN
+F 2 "Resistor_SMD:R_0603_1608Metric" V 5930 6400 50  0001 C CNN
+F 3 "~" H 6000 6400 50  0001 C CNN
+	1    6000 6400
+	0    1    1    0
+$EndComp
+$Comp
+L Device:R R50
+U 1 1 5CAD694E
+P 6000 8500
+F 0 "R50" V 6100 8400 50  0000 C CNN
+F 1 "4.7" V 6100 8600 50  0000 C CNN
+F 2 "Resistor_SMD:R_0603_1608Metric" V 5930 8500 50  0001 C CNN
+F 3 "~" H 6000 8500 50  0001 C CNN
+	1    6000 8500
+	0    1    1    0
+$EndComp
+$Comp
+L Device:R R51
+U 1 1 5CAD6A66
+P 6000 8700
+F 0 "R51" V 6100 8600 50  0000 C CNN
+F 1 "4.7" V 6100 8800 50  0000 C CNN
+F 2 "Resistor_SMD:R_0603_1608Metric" V 5930 8700 50  0001 C CNN
+F 3 "~" H 6000 8700 50  0001 C CNN
+	1    6000 8700
+	0    1    1    0
+$EndComp
+Wire Wire Line
+	6150 8500 6250 8500
+Wire Wire Line
+	6150 8700 6700 8700
+Wire Wire Line
+	5850 8500 5750 8500
+Wire Wire Line
+	5750 8700 5850 8700
+Wire Wire Line
+	5750 6200 5850 6200
+Wire Wire Line
+	5750 6400 5850 6400
+Wire Wire Line
+	6150 6200 6250 6200
+Wire Wire Line
+	6150 6400 6700 6400
+Text Label 21050 8800 2    50   ~ 0
+CAN0_L
+Text Label 11850 11800 2    50   ~ 0
+CAN0_L
+Wire Wire Line
+	11250 11800 11850 11800
+Wire Wire Line
+	11250 11500 11850 11500
+Text Label 11850 11500 2    50   ~ 0
+CAN0_H
+Wire Wire Line
+	11200 13150 11800 13150
+Wire Wire Line
+	11200 13450 11800 13450
+Text Label 11800 13150 2    50   ~ 0
+CAN1_H
+Text Label 11800 13450 2    50   ~ 0
+CAN1_L
+Text Label 21050 8900 2    50   ~ 0
+CAN0_H
+Text Label 21050 9000 2    50   ~ 0
+CAN1_L
+Text Label 21050 9100 2    50   ~ 0
+CAN1_H
 $EndSCHEMATC
